File: Variable Buck Converter.kicad_pcb (KiCad board)
At the start: 4 copper layers, 52.2 x 88.4 mm, 63 parts, among them IC1 SN74LVC2G17DBVR, IC2 LMG1210RVRT, J1 EN/PWM Header, J2 Vin_Terminal, J3 VSUPPLY_Terminal, J4 Inductor, J5 Output_Terminal, J6 RASPI Socket 1, J7 RASPI Socket 2, Q1 EPC2001C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

Commit message: v1.1.0 Gerber
Parts:
- added D4: LED, LED_SMD:LED_0603_1608Metric, F.Cu at (116.4, 67.3)
- added R15: 100K, Resistor_SMD:R_0603_1608Metric, F.Cu at (116.4, 70.6)
- added R16: 0.01R, Resistor_SMD:R_1206_3216Metric, F.Cu at (121.7, 97.9)
- added TP14: TestPoint_Probe, TestPoint:TestPoint_Loop_D2.60mm_Drill1.6mm_Beaded, F.Cu at (118.4, 102.2)
- added TP15: TestPoint_Probe, TestPoint:TestPoint_Loop_D2.60mm_Drill1.6mm_Beaded, F.Cu at (125.2, 102.2)
- J2: value Vin_Terminal -> Vin_IC
- J3: value VSUPPLY_Terminal -> Vin_Buck
- moved TP3 3.98 mm to (119.3, 94.4)
- moved Q1 2.21 mm to (113.8, 92.2)
- moved Q2 2.18 mm to (113.8, 96.5)
- moved TP8 1.73 mm to (107.6, 89.0)
- moved R12 0.79 mm to (108.6, 96.1)
- moved R11 0.79 mm to (108.6, 92.8)
- moved TP9 0.50 mm to (109.4, 100.3)
- moved C7 0.10 mm to (103.7, 99.9)
Connections:
- net Net-(J3-Pin_1) renamed +Vin_Buck
- J4 pad 1: /Buck Converter/HS -> Net-(J4-Pin_1)
Routing:
- net /Buck Converter/HS: track 5.06 -> 10.1 mm, vias 8 -> 9
- net Net-(D4-A): track 0.00 -> 1.72 mm
- net /Buck Converter/LO: track 8.24 -> 7.26 mm
- net /Buck Converter/HO: track 6.94 -> 6.27 mm
- net GND: vias 95 -> 100
- added copper zone on F.Cu, net Net-(J4-Pin_1)
Other:
- board text added: "V_IN : IC"
- board text added: "V_INPUT : BUCK"
- board text added: "V_OUT : BUCK"
- board text removed: "V_INPUT"
- board text removed: "V_OUT"
- board text removed: "V_SUPPLY"

Commit message: C14 change, BoM and CPL
Parts:
- C14: footprint Capacitor_SMD:C_1206_3216Metric -> Capacitor_SMD:CP_Elec_6.3x5.9
- moved C8 3.76 mm to (123.9, 90.0)
- moved C11 3.33 mm to (123.9, 91.7)
- moved C14 1.94 mm to (123.9, 85.5)
- moved R14 0.62 mm to (127.2, 79.6)
