File: Variable Buck Converter.kicad_sch (KiCad schematic)
At the start: 8 parts, among them J6 RASPI Socket 1, J7 RASPI Socket 2, U1 Pico

Commit message: C14 change, BoM and CPL
Parts:
- C1: Manufacturer_Part_Number (none) -> CL10A106MA8NRNC
- C2: Manufacturer_Part_Number (none) -> CL10B104JB8NNND
- J6, J7: Manufacturer_Part_Number (none) -> PH1-20-UA
- JP1: Manufacturer_Part_Number (none) -> HTSW-102-07-T-S
- R1: Manufacturer_Part_Number (none) -> RT0603BRD0791KL
- R2: Manufacturer_Part_Number (none) -> RT0603BRD0718KL
- U1: now not fitted
Changed lines of the file:
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@@
+			)
+		)
+		(property "Manufacturer_Part_Number" "CL10B104JB8NNND"
+			(at 144.78 106.68 0)
+			(effects
+				(font
+					(size 1.27 1.27)
+				)
+				(hide yes)
 			)
 		)
@@
 			)
 		)
+		(property "Manufacturer_Part_Number" "HTSW-102-07-T-S"
+			(at 125.73 82.55 0)
+			(effects
+				(font
+					(size 1.27 1.27)
+				)
+				(hide yes)
+			)
+		)
 		(pin "1"
 		)
@@
 		(in_bom no)
 		(on_board no)
-		(dnp no)
+		(dnp yes)
 		(fields_autoplaced yes)
 		(property "Reference" "U1"
@@
 		)
 		(property "Description" "Resistor"
+			(at 157.48 109.22 0)
+			(effects
+				(font
+					(size 1.27 1.27)
+				)
+				(hide yes)
+			)
+		)
+		(property "Manufacturer_Part_Number" "RT0603BRD0718KL"
 			(at 157.48 109.22 0)
 			(effects
@@
 			)
 		)
+		(property "Manufacturer_Part_Number" "PH1-20-UA"
+			(at 109.22 105.41 0)
+			(effects
+				(font
+					(size 1.27 1.27)
+				)
+				(hide yes)
+			)
+		)
 		(pin "4"
 		)
@@
 			)
 		)
+		(property "Manufacturer_Part_Number" "CL10A106MA8NRNC"
+			(at 116.84 68.58 0)
+			(effects
+				(font
+					(size 1.27 1.27)
+				)
+				(hide yes)
+			)
+		)
 		(pin "2"
 		)
@@
 			)
 		)
+		(property "Manufacturer_Part_Number" "RT0603BRD0791KL"
+			(at 157.48 96.52 0)
+			(effects
+				(font
+					(size 1.27 1.27)
+				)
+				(hide yes)
+			)
+		)
 		(pin "1"
 		)
@@
 			(at 63.5 105.41 0)
 			(effects
+				(font
+					(size 1.27 1.27)
+				)
+				(hide yes)
+			)
+		)
+		(property "Manufacturer_Part_Number" "PH1-20-UA"
+			(at 63.5 105.41 0)
+			(effects
