File: buck_converter.kicad_sch (KiCad schematic)
At the start: 56 parts, among them IC1 SN74LVC2G17DBVR, IC2 LMG1210RVRT, J1 EN/PWM Header, J2 Vin_Terminal, J3 VSUPPLY_Terminal, J4 Inductor, J5 Output_Terminal, Q1 EPC2001C, Q2 EPC2001C

Commit message: v1.1.0 Gerber
Parts:
- added D4: LED, LED_SMD:LED_0603_1608Metric, symbol Device:LED
- added R15: 100K, Resistor_SMD:R_0603_1608Metric, symbol Device:R
- added R16: 0.01R, Resistor_SMD:R_1206_3216Metric, symbol Device:R
- added TP14, TP15: TestPoint_Probe, TestPoint:TestPoint_Loop_D2.60mm_Drill1.6mm_Beaded, symbol Connector:TestPoint_Probe
- J2: value Vin_Terminal -> Vin_IC
- J3: value VSUPPLY_Terminal -> Vin_Buck
Connections:
- net GND: now also D4.1 (K)
- net HS: now also R16.1, TP14.1; no longer J4.1 (Pin_1)
- net +Vin_Buck: now reaches J3.1 (Pin_1), JP6.2 (B), R13.2, TP10.1
- net +Vin_Buck: now also R15.1
- new net: D4.2 (A), R15.2
- new net: J4.1 (Pin_1), R16.2, TP15.1
Other:
- moved on the sheet: C11, C14, C8, J4, J5, Q1, Q2, R11, R12, R14, TP12, TP13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

Commit message: C14 change, BoM and CPL
Parts:
- C10, C11, C3, C9: Manufacturer_Part_Number (none) -> CL10B104JB8NNND
- C12, C13, C5, C6, C8: Manufacturer_Part_Number (none) -> CL10A106MA8NRNC
- C14: footprint Capacitor_SMD:C_1206_3216Metric -> Capacitor_SMD:CP_Elec_6.3x5.9; Manufacturer_Part_Number (none) -> 865080545012
- C4, C7: Manufacturer_Part_Number (none) -> YFF18PW0J474MT0H0N
- D2, D3, D4: Manufacturer_Part_Number (none) -> LTST-C190GKT
- J1: Manufacturer_Part_Number (none) -> PH1-04-UA
- J2, J3, J4, J5: Manufacturer_Part_Number (none) -> 1548128
- JP2, JP3, JP5, JP6: Manufacturer_Part_Number (none) -> HTSW-102-07-T-S
- JP4: Manufacturer_Part_Number (none) -> PH1-03-UA; now in the parts list
- POT1, POT2: Manufacturer_Part_Number (none) -> 3296W-1-105LF
- R10, R3, R4, R9: Manufacturer_Part_Number (none) -> RT0603FRE0720KL
- R11, R12, R5, R6: Manufacturer_Part_Number (none) -> RCG06030000Z0EA
- R13, R14, R16: Manufacturer_Part_Number (none) -> PE1206DRM7W0R01L
- R15, R8: Manufacturer_Part_Number (none) -> RT0603FRE07100KL
- R7: Manufacturer_Part_Number (none) -> RT0603FRE131KL
- TP1, TP2, TP5: Manufacturer_Part_Number (none) -> 5278
- TP10, TP11, TP6, TP7: Manufacturer_Part_Number (none) -> 5270
- TP12, TP13: Manufacturer_Part_Number (none) -> 5274
- TP14, TP15: Manufacturer_Part_Number (none) -> 5277
- TP3, TP4: Manufacturer_Part_Number (none) -> 5271
- TP8, TP9: Manufacturer_Part_Number (none) -> 5273
